Commit message: world_ur and pi rotation fixes

File: urdf/ur.urdf.xacro (robot description, xacro)
@@ -52,5 +52,5 @@
    <xacro:property name="is_sim_ignition" value="$(arg sim_ignition)"/>
    <!-- create link fixed to the "world" -->
-   <link name="world" />
+   <link name="world_ur" />
    <xacro:if value="${is_sim_gazebo or is_sim_ignition}">
      <link name="ground_plane">
@@ -73,5 +73,5 @@
      <joint name="ground_plane_joint" type="fixed">
        <origin xyz="0 0 -0.01" rpy="0 0 0"/>
-       <parent link="world"/>
+       <parent link="world_ur"/>
        <child link="ground_plane"/>
      </joint>
@@ -81,5 +81,5 @@
      name="$(arg name)"
      tf_prefix="$(arg tf_prefix)"
-     parent="world"
+     parent="world_ur"
      joint_limits_parameters_file="$(arg joint_limit_params)"
      kinematics_parameters_file="$(arg kinematics_params)"
@@ -119,5 +119,5 @@
    <xacro:if value="$(arg sim_gazebo)">
     <!-- Gazebo plugins -->
-    <gazebo reference="world">
+    <gazebo reference="world_ur">
     </gazebo>
     <gazebo>
@@ -129,5 +129,5 @@
   <xacro:if value="$(arg sim_ignition)">
     <!-- Gazebo plugins -->
-    <gazebo reference="world">
+    <gazebo reference="world_ur">
     </gazebo>
     <gazebo>

File: urdf/ur_macro.xacro (robot description, xacro)
@@ -135,5 +135,6 @@
     <link name="${tf_prefix}base_link_inertia">
       <visual>
-        <origin xyz="0 0 0" rpy="0 0 ${pi}"/>
+        <!-- <origin xyz="0 0 0" rpy="0 0 ${pi}"/> -->
+        <origin xyz="0 0 0" rpy="0 0 0" />
         <geometry>
           <xacro:get_mesh name="base" type="visual"/>
@@ -141,5 +142,6 @@
       </visual>
       <collision>
-        <origin xyz="0 0 0" rpy="0 0 ${pi}"/>
+        <!-- <origin xyz="0 0 0" rpy="0 0 ${pi}"/> -->
+        <origin xyz="0 0 0" rpy="0 0 0" />
         <geometry>
           <xacro:get_mesh name="base" type="collision"/>
@@ -329,5 +331,6 @@
            link/frame) to introduce the necessary rotation over Z (of pi rad).
       -->
-      <origin xyz="0 0 0" rpy="0 0 ${pi}" />
+      <!-- <origin xyz="0 0 0" rpy="0 0 ${pi}" /> -->
+      <origin xyz="0 0 0" rpy="0 0 0" />
     </joint>
     <joint name="${tf_prefix}shoulder_pan_joint" type="revolute">
